Commit message: dsa

File: catkin_ws/src/my_robot/urdf/dif_robot.xacro (robot description, xacro)
@@ -1,106 +1,234 @@
 <?xml version="1.0"?>
-<robot name="diffbot" xmlns:xacro="http://ros.org/wiki/xacro">
-  <xacro:property name="wheel_radius" value="0.05"/>
-  <xacro:property name="wheel_width" value="0.02"/>
-  <xacro:property name="base_length" value="0.4"/>
-  <xacro:property name="base_width"  value="0.3"/>
-  <!-- Base -->
+<robot name="differential_wheeled_robot" xmlns:xacro="http://www.ros.org/wiki/xacro">
+  <xacro:include filename="$(find my_robot)/urdf/wheel.urdf.xacro" />
+<!-- Defining the colors used in this robot -->
+  <material name="Black">
+    <color rgba="0.0 0.0 0.0 1.0"/>
+  </material>
+  <material name="Red">
+    <color rgba="0.8 0.0 0.0 1.0"/>
+  </material>
+  <material name="White">
+    <color rgba="1.0 1.0 1.0 1.0"/>
+  </material>
+  <material name="Blue">
+    <color rgba="0.0 0.0 0.8 1.0"/>
+  </material>
+  <!-- PROPERTY LIST -->
+  <!--All units in m-kg-s-radians unit system -->
+  <property name="M_PI" value="3.1415926535897931" />
+  <property name="M_PI_2" value="1.570796327" />
+  <property name="DEG_TO_RAD" value="0.017453293" />
+  <!-- Main body radius and height -->
+  <!-- Main Body Cylinder base   -->
+  <property name="base_height" value="0.02" />
+  <property name="base_radius" value="0.15" />
+  <property name="base_mass" value="5" /> <!-- in kg-->
+  <!-- caster wheel radius and height -->
+  <!-- caster wheel mass -->
+  <property name="caster_f_height" value="0.04" />
+  <property name="caster_f_radius" value="0.025" />
+  <property name="caster_f_mass" value="0.5" /> <!-- in kg-->
+  <!-- caster wheel radius and height -->
+  <!-- caster wheel mass -->
+  <property name="caster_b_height" value="0.04" />
+  <property name="caster_b_radius" value="0.025" />
+  <property name="caster_b_mass" value="0.5" /> <!-- in kg-->
+  <!-- Wheels -->
+  <property name="wheel_mass" value="2.5" /> <!-- in kg-->
+  <property name="base_x_origin_to_wheel_origin" value="0.25" />
+  <property name="base_y_origin_to_wheel_origin" value="0.3" />
+  <property name="base_z_origin_to_wheel_origin" value="0.0" />
+  <!-- Hokuyo Laser scanner -->
+  <property name="hokuyo_size" value="0.05" />
+  <!-- Macro for calculating inertia of cylinder -->
+  <macro name="cylinder_inertia" params="m r h">
+    <inertia  ixx="${m*(3*r*r+h*h)/12}" ixy = "0" ixz = "0"
+              iyy="${m*(3*r*r+h*h)/12}" iyz = "0"
+              izz="${m*r*r/2}" />
+  </macro>
+  <!-- BASE-FOOTPRINT -->
+  <!-- base_footprint is a fictitious link(frame) that is on the ground right below base_link origin -->
+  <link name="base_footprint">
+    <inertial>
+      <mass value="0.0001" />
+      <origin xyz="0 0 0" />
+      <inertia ixx="0.0001" ixy="0.0" ixz="0.0"
+          iyy="0.0001" iyz="0.0"
+          izz="0.0001" />
+    </inertial>
+    <visual>
+        <origin xyz="0 0 0" rpy="0 0 0" />
+        <geometry>
+            <box size="0.001 0.001 0.001" />
+        </geometry>
+    </visual>
+  </link>
+  <gazebo reference="base_footprint">
+    <turnGravityOff>false</turnGravityOff>
+  </gazebo>
+  <joint name="base_footprint_joint" type="fixed">
+    <origin xyz="0 0 ${wheel_radius - base_z_origin_to_wheel_origin}" rpy="0 0 0" />
+    <parent link="base_footprint"/>
+    <child link="base_link" />
+  </joint>
+  <!-- BASE-LINK -->
+  <!--Actual body/chassis of the robot-->
   <link name="base_link">
-    <visual>
-      <geometry>
-        <box size="${base_length} ${base_width} 0.1"/>
-      </geometry>
-      <origin xyz="0 0 0.05"/>
+    <inertial>
+      <mass value="${base_mass}" />
+      <origin xyz="0 0 0" />
+      <!--The 3x3 rotational inertia matrix. -->
+        <cylinder_inertia  m="${base_mass}" r="${base_radius}" h="${base_height}" />
+    </inertial>
+    <visual>
+      <origin xyz="0 0 0" rpy="0 0 0" />
+      <geometry>
+          <cylinder length="${base_height}" radius="${base_radius}" />
+      </geometry>
+      <material name="White" />
     </visual>
     <collision>
-      <geometry>
-        <box size="${base_length} ${base_width} 0.1"/>
-      </geometry>
-      <origin xyz="0 0 0.05"/>
+      <origin xyz="0 0 0" rpy="0 0 0 " />
+      <geometry>
+          <cylinder length="${base_height}" radius="${base_radius}" />
+      </geometry>
     </collision>
-    <inertial>
-      <mass value="10"/>
-      <inertia
-        ixx="0.1" ixy="0.0" ixz="0.0"
-        iyy="0.1" iyz="0.0" izz="0.1"/>
-      </inertial>
   </link>
-  <!-- Wheels -->
-  <xacro:macro name="wheel" params="side x_pos">
-    <link name="${side}_wheel">
-      <visual>
-        <geometry>
-          <cylinder radius="${wheel_radius}" length="${wheel_width}"/>
-        </geometry>
-        <origin rpy="0 1.5708 0"/>
-      </visual>
+  <gazebo reference="base_link">
+    <material>Gazebo/White</material>
+    <turnGravityOff>false</turnGravityOff>
+  </gazebo>
+<!--Caster front  -->
+    <link name="caster_front_link">
+    <visual>
+      <origin xyz="0 0.02 0" rpy="${M_PI/2} 0 0" />
+      <geometry>
+	<sphere radius="${caster_f_radius}" />
+      </geometry>
+      <material name="Black" />
+    </visual>
       <collision>
         <geometry>
-          <cylinder radius="${wheel_radius}" length="${wheel_width}"/>
+	<sphere radius="${caster_f_radius}" />
         </geometry>
-        <origin rpy="0 1.5708 0"/>
+      <origin xyz="0 0.02 0" rpy="${M_PI/2} 0 0" />
       </collision>
       <inertial>
-        <mass value="1"/>
-        <inertia
-          ixx="0.01" ixy="0.0" ixz="0.0"
-          iyy="0.01" iyz="0.0" izz="0.01"/>
-        </inertial>
+        <mass value="${caster_f_mass}" />
+        <origin xyz="0 0 0" />
+        <inertia ixx="0.001" ixy="0.0" ixz="0.0"
+                 iyy="0.001" iyz="0.0"
+                 izz="0.001" />
+      </inertial>
     </link>
-    <joint name="${side}_wheel_joint" type="continuous">
+ <joint name="caster_front_joint" type="fixed">
       <parent link="base_link"/>
-      <child link="${side}_wheel"/>
-      <origin xyz="${x_pos} ${'0.15' if side == 'left' else '-0.15'} 0.05"/>
-      <axis xyz="0 0 1"/>
+      <child link="caster_front_link"/>
+      <origin xyz="0.115 0.0 0.007" rpy="${-M_PI/2} 0 0"/>
     </joint>
-  </xacro:macro>
-  <xacro:wheel side="left" x_pos="0"/>
-  <xacro:wheel side="right" x_pos="0"/>
-  <!-- Camera -->
-  <link name="camera_link">
-    <visual>
-      <geometry><box size="0.05 0.05 0.05"/></geometry>
+  <gazebo reference="caster_front_link">
+    <turnGravityOff>false</turnGravityOff>
+  </gazebo>
+<!--Caster back  -->
+    <link name="caster_back_link">
+    <visual>
+      <origin xyz="0.02 0.02 0 " rpy="${M_PI/2} 0 0" />
+      <geometry>
+	<sphere radius="${caster_b_radius}" />
+      </geometry>
+      <material name="Black" />
+    </visual>
+      <collision>
+        <geometry>
+		<sphere radius="${caster_b_radius}" />
+        </geometry>
+      <origin xyz="0 0.02 0 " rpy="${M_PI/2} 0 0" />
+      </collision>
+      <inertial>
+        <mass value="${caster_b_mass}" />
+        <origin xyz="0 0 0" />
+        <inertia ixx="0.001" ixy="0.0" ixz="0.0"
+                 iyy="0.001" iyz="0.0"
+                 izz="0.001" />
+      </inertial>
+    </link>
+    <joint name="caster_back_joint" type="fixed">
+      <parent link="base_link"/>
+      <child link="caster_back_link"/>
+      <origin xyz="-0.135 0.0 0.009" rpy="${-M_PI/2} 0 0"/>
+    </joint>
+  <gazebo reference="caster_back_link">
+    <turnGravityOff>false</turnGravityOff>
+  </gazebo>
+<!-- Wheel Definitions -->
+  <wheel fb="front" lr="right" parent="base_link" translateX="0" translateY="0.5" flipY="1"/>
+  <wheel fb="front" lr="left" parent="base_link" translateX="0" translateY="-0.5" flipY="1"/>
+  <!-- SENSORS -->
+  <!-- hokuyo -->
+  <link name="hokuyo_link">
+    <visual>
+      <origin xyz="0 0 0" rpy="0 0 0" />
+      <geometry>
+        <box size="${hokuyo_size} ${hokuyo_size} ${hokuyo_size}"/>
+      </geometry>
+      <material name="Blue" />
     </visual>
   </link>
-  <joint name="camera_joint" type="fixed">
+  <joint name="hokuyo_joint" type="fixed">
+    <origin xyz="${base_radius - hokuyo_size/2} 0 ${base_height+hokuyo_size/4}" rpy="0 0 0" />
     <parent link="base_link"/>
-    <child link="camera_link"/>
-    <origin xyz="0.1 0 0.2" rpy="0 0 0"/>
+    <child link="hokuyo_link" />
   </joint>
-  <!-- Lidar -->
-  <link name="lidar_link">
-    <visual>
-      <geometry><cylinder radius="0.03" length="0.05"/></geometry>
-      <origin rpy="0 0 0"/>
-    </visual>
-  </link>
-  <joint name="lidar_joint" type="fixed">
-    <parent link="base_link"/>
-    <child link="lidar_link"/>
-    <origin xyz="0 0 0.15"/>
-  </joint>
-  <!-- Plugins -->
+  <gazebo reference="hokuyo_link">
+    <material>Gazebo/Blue</material>
+    <turnGravityOff>false</turnGravityOff>
+    <sensor type="ray" name="head_hokuyo_sensor">
+      <pose>${hokuyo_size/2} 0 0 0 0 0</pose>
+      <visualize>false</visualize>
+      <update_rate>40</update_rate>
+      <ray>
+        <scan>
+          <horizontal>
+            <samples>720</samples>
+            <resolution>1</resolution>
+            <min_angle>-1.570796</min_angle>
+            <max_angle>1.570796</max_angle>
+          </horizontal>
+        </scan>
+        <range>
+          <min>0.10</min>
+          <max>10.0</max>
+          <resolution>0.001</resolution>
+        </range>
+      </ray>
+      <plugin name="gazebo_ros_head_hokuyo_controller" filename="libgazebo_ros_laser.so">
+        <topicName>/scan</topicName>
+        <frameName>hokuyo_link</frameName>
+      </plugin>
+    </sensor>
+  </gazebo>
+  <!-- Differential drive controller  -->
   <gazebo>
-    <plugin name="diff_drive_controller" filename="libgazebo_ros_diff_drive.so">
-      <left_wheel>left_wheel</left_wheel>
-      <right_wheel>right_wheel</right_wheel>
-      <wheel_separation>0.3</wheel_separation>
-      <wheel_diameter>0.1</wheel_diameter>
-      <robot_base_frame>base_link</robot_base_frame>
-      <updateRate>50</updateRate>
+    <plugin name="differential_drive_controller" filename="libgazebo_ros_diff_drive.so">
+      <rosDebugLevel>Debug</rosDebugLevel>
+      <publishWheelTF>false</publishWheelTF>
+      <robotNamespace>/</robotNamespace>
+      <publishTf>1</publishTf>
+      <publishWheelJointState>false</publishWheelJointState>
+      <alwaysOn>true</alwaysOn>
+      <updateRate>100.0</updateRate>
+      <leftJoint>front_left_wheel_joint</leftJoint>
+      <rightJoint>front_right_wheel_joint</rightJoint>
+      <wheelSeparation>${2*base_radius}</wheelSeparation>
+      <wheelDiameter>${2*wheel_radius}</wheelDiameter>
+      <broadcastTF>1</broadcastTF>
+      <wheelTorque>30</wheelTorque>
+      <wheelAcceleration>1.8</wheelAcceleration>
       <commandTopic>cmd_vel</commandTopic>
+      <odometryFrame>odom</odometryFrame>
       <odometryTopic>odom</odometryTopic>
+      <robotBaseFrame>base_footprint</robotBaseFrame>
     </plugin>
-    <plugin name="camera_controller" filename="libgazebo_ros_camera.so">
-      <alwaysOn>true</alwaysOn>
-      <cameraName>robot_camera</cameraName>
-      <imageTopicName>camera/image_raw</imageTopicName>
-      <cameraInfoTopicName>camera/camera_info</cameraInfoTopicName>
-      <frameName>camera_link</frameName>
-    </plugin>
-    <plugin name="lidar_controller" filename="libgazebo_ros_laser.so">
-      <topicName>scan</topicName>
-      <frameName>lidar_link</frameName>
-    </plugin>
   </gazebo>
 </robot>

File: catkin_ws/src/my_robot/urdf/mob_rob.urdf (robot description, URDF)
Before this commit: robot diffbot, 5 links, 4 joints
Links:
- removed link base_link
- removed link camera_link
- removed link left_wheel
- removed link lidar_link
- removed link right_wheel
- added link body_link, mass 10; collision box size=1.0 0.6 0.3; visual box size=1.0 0.6 0.3
- added link wheel1_link, mass 1; collision cylinder length=0.1 radius=0.15; visual cylinder length=0.1 radius=0.15
- added link world
Joints:
- removed joint camera_joint
- removed joint left_wheel_joint
- removed joint lidar_joint
- removed joint right_wheel_joint
- added joint base_joint: type fixed, parent world, child body_link, origin xyz=0 0 0 rpy=0 0 0
- added joint wheel1_joint: type continuous, parent body_link, child wheel1_link, origin xyz=-0.3 -0.35 0 rpy=0 0 0, axis 0 1 0

File: catkin_ws/src/my_robot/urdf/simple_robot.urdf (robot description, URDF)
Before this commit: robot simple_robot, 3 links, 2 joints
Links:
- link base_link: geometry collision box size=1 1 1; visual box size=0.3 0.3 0.1
